File: thingamaPRO_main/procon_gcc_main_pcb.kicad_sch (KiCad schematic)
At the start: 82 parts, among them J1 Rumble, J3 To Button Board, J4 Conn_01x06_Female, J5 Conn_01x02, J6 Conn_01x03_Male, J7 Rumble, J9 USB_C_Receptacle, Q1 Q_PMOS_GDS, Q2 Q_NMOS_GSD, Q3 Q_NMOS_GSD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

Commit message: Matrix Rewire for front boards
Swapped from direct to a matrix layout to support oem front boards
Parts:
- removed J?: To Button Board, procon_gcc:molex_5051101492_14P, symbol Connector_Generic:Conn_01x14
Connections:
- net +3V3: now also J3.2 (Pin_2)
- net BTN_A: no longer J3.1 (Pin_1), U15.28 (GPIO17)
- net BTN_B: no longer J3.2 (Pin_2), U15.27 (GPIO16)
- net BTN_DP_D: no longer J3.11 (Pin_11), U15.13 (GPIO10)
- net BTN_DP_L: no longer J3.12 (Pin_12), U15.11 (GPIO8)
- net BTN_DP_R: no longer J3.13 (Pin_13), U15.14 (GPIO11)
- net BTN_DP_U: no longer J3.10 (Pin_10), U15.12 (GPIO9)
- net BTN_LT: no longer J3.8 (Pin_8), U15.34 (GPIO22)
- net BTN_RT: no longer J3.9 (Pin_9), U15.32 (GPIO21)
- net BTN_ST: no longer J3.5 (Pin_5), U15.7 (GPIO5)
- net BTN_X: no longer J3.3 (Pin_3), U15.29 (GPIO18)
- net BTN_Y: no longer J3.4 (Pin_4), U15.30 (GPIO19)
- net BTN_ZL: no longer J3.6 (Pin_6), U15.16 (GPIO13)
- net BTN_ZR: no longer D4.2 (A), J3.7 (Pin_7), U15.31 (GPIO20)
- net GND: now also J3.1 (Pin_1), J3.12 (Pin_12); no longer J3.14 (Pin_14)
- new net Ddown: U15.13 (GPIO10)
- new net Dleft: U15.11 (GPIO8)
- new net Dright: U15.14 (GPIO11)
- new net Dup: U15.12 (GPIO9)
- new net LED_EN: J3.3 (Pin_3)
- new net NFC: J3.13 (Pin_13), J3.14 (Pin_14)
- new net Push_A: J3.4 (Pin_4), U15.16 (GPIO13)
- new net Push_B: J3.6 (Pin_6), U15.28 (GPIO17)
- new net Push_C: D4.2 (A), J3.9 (Pin_9), U15.31 (GPIO20)
- new net Push_D: J3.10 (Pin_10), U15.32 (GPIO21)
- new net Scan_A: J3.11 (Pin_11), U15.34 (GPIO22)
- new net Scan_B: J3.8 (Pin_8), U15.30 (GPIO19)
- new net Scan_C: J3.5 (Pin_5), U15.27 (GPIO16)
- new net Scan_D: J3.7 (Pin_7), U15.29 (GPIO18)
- new net Start: U15.7 (GPIO5)
