File: progcc_v3_main/procon_gcc_main_pcb.kicad_pcb (KiCad board)
At the start: 4 copper layers, 110.9 x 59.5 mm, 73 parts, among them J1 Rumble, J3 To Button Board, J4 Conn_01x06_Female, J6 Conn_01x03_Male, J7 Rumble, J9 USB_C_Receptacle, Q1 Q_PMOS_GDS, Q2 Q_PMOS_GDS, Q3 Q_PMOS_GDS, Q4 BSS138, Q5 BSS138, Q6 BSS138, SW1 GL18_SW, SW2 GL18_SW, SW3 TS09-63-25-R-260-SMT, U1 GH39F (Hall SOT23), U14 XC6206PxxxMR, U2 GH39F (Hall SOT23), U3 GH39F (Hall SOT23), U4 GH39F (Hall SOT23), U5 GL16112, U6 RP2040, U9 W25Q128JVS, Y1 Crystal_GND3

Commit message: some schematic fixes+some positioning
Parts:
- removed J7: Rumble, Connector_PinHeader_2.00mm:PinHeader_1x02_P2.00mm_Horizontal
- added C16: 1u, Capacitor_SMD:C_0603_1608Metric, F.Cu at (154.4, 150.5)
- added C17: 1u, Capacitor_SMD:C_0603_1608Metric, F.Cu at (92.5, 129.2)
- added C18: 1u, Capacitor_SMD:C_0603_1608Metric, F.Cu at (169.3, 142.7)
- added C19: 1u, Capacitor_SMD:C_0603_1608Metric, F.Cu at (107.9, 121.8)
- added J2: Rumble, progcc_v3:rumble_pins, F.Cu at (179.8, 142.8)
- added U7: MCP3002, progcc_v3:SOIC-8_3.9x4.9mm_P1.27mm, F.Cu at (119.6, 117.5)
- added U8: MCP3002, progcc_v3:SOIC-8_3.9x4.9mm_P1.27mm, F.Cu at (147.5, 124.4)
- C12, C14, C15, C8: value 1u -> .047u
- J1: footprint Connector_PinHeader_2.00mm:PinHeader_1x02_P2.00mm_Horizontal -> progcc_v3:rumble_pins
- J4: footprint Connector_PinHeader_2.00mm:PinHeader_1x06_P2.00mm_Horizontal -> progcc_v3:GCC_Header_Straight_1x06_Pitch2.00mm
- J6: footprint Connector_PinHeader_2.00mm:PinHeader_1x03_P2.00mm_Horizontal -> progcc_v3:PinHeader_1x03_P2.54mm_Vertical
- R14, R19, R29, R30: footprint Resistor_SMD:R_0603_1608Metric_Pad0.98x0.95mm_HandSolder -> Resistor_SMD:R_0402_1005Metric
- moved SW3 135.3 mm to (164.2, 113.8), turned to 90 degrees
- moved C14 119.3 mm to (165.8, 148.9), turned to 180 degrees
- moved D3 109.5 mm to (141.2, 105.4), turned to 90 degrees
- moved F2 98.0 mm to (125.8, 107.2)
- moved C4 77.0 mm to (142.7, 105.4), turned to 90 degrees
- moved F3 72.1 mm to (129.3, 86.6)
- moved R11 71.4 mm to (103.4, 88.9), turned to 180 degrees
- moved R13 70.2 mm to (105.4, 99.8)
- moved Q4 68.0 mm to (99.6, 88.9)
- moved R6 62.2 mm to (97.5, 91.4)
- moved D4 60.7 mm to (103.9, 102.9)
- moved C12 59.0 mm to (113.8, 119.3), turned to -90 degrees
- moved Q5 56.4 mm to (80.8, 88.6)
- moved C15 56.3 mm to (160.5, 130.2), turned to -90 degrees
- moved C8 53.9 mm to (104.2, 130.1), turned to -90 degrees
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Connections:
- net RUMBLE+ renamed +5V
- C12 pad 1: +3.3V -> GND
- C12 pad 2: GND -> LY
- C14 pad 1: +3.3V -> GND
- C14 pad 2: GND -> RX
- C15 pad 1: +3.3V -> GND
- C15 pad 2: GND -> RY
- C8 pad 1: +3.3V -> GND
- C8 pad 2: GND -> LX
- J9 pad S1: GND -> unconnected-(J9-PadS1)
- SW1 pad S2: LS_BUTTON -> GND
- SW1 pad S3: GND -> LS_BUTTON
- SW2 pad S2: RS_BUTTON -> GND
- SW2 pad S3: GND -> RS_BUTTON
Routing:
- net +3.3V: track 51.2 -> 21.2 mm
- net RX: track 3.83 -> 33.6 mm
- net Net-(R17-Pad1): track 33.6 -> 3.83 mm
- net LX: track 3.88 -> 30.0 mm
- net (no net): track 23.7 -> 0.00 mm
- net RY: track 3.76 -> 26.0 mm
- net Net-(R18-Pad1): track 26.0 -> 3.76 mm
- net Net-(R16-Pad1): track 12.1 -> 3.48 mm
- net LY: track 3.48 -> 12.1 mm
- net +1V1: track 26.0 -> 18.6 mm
- net +3.3V_PRE: track 0.00 -> 5.32 mm
- net Net-(R29-Pad2): track 0.00 -> 3.91 mm
- net Net-(R15-Pad1): track 0.00 -> 3.88 mm
- net Net-(R30-Pad2): track 0.00 -> 3.51 mm
- net XTAL_OUT: track 4.26 -> 1.51 mm, vias 1 -> 0
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
Commit message: Schematic finalization
Parts:
- removed J1, J2: Rumble, progcc_v3:rumble_pins
- removed J6: Conn_01x03_Male, progcc_v3:PinHeader_1x03_P2.54mm_Vertical
- removed U14: XC6206PxxxMR, Package_TO_SOT_SMD:SOT-23
- added C20: 100n, Capacitor_SMD:C_0402_1005Metric, F.Cu at (35.6, 147.3)
- added C21: 100n, Capacitor_SMD:C_0402_1005Metric, F.Cu at (38.4, 147.3)
- added C23: 100n, Capacitor_SMD:C_0402_1005Metric, F.Cu at (41.3, 147.3)
- added L1: SK6805-EC-15, progcc_v3:SK6805-EC-15, F.Cu at (44.8, 136.3)
- added L2: SK6805-EC-15, progcc_v3:SK6805-EC-15, F.Cu at (44.8, 132.5)
- added L3: SK6805-EC-15, progcc_v3:SK6805-EC-15, F.Cu at (27.5, 141.8)
- added L4: SK6805-EC-15, progcc_v3:SK6805-EC-15, F.Cu at (48.6, 136.3)
- added L5: SK6805-EC-15, progcc_v3:SK6805-EC-15, F.Cu at (36.4, 144.1)
- added L6: SK6805-EC-15, progcc_v3:SK6805-EC-15, F.Cu at (41.5, 140.1)
- added L7: SK6805-EC-15, progcc_v3:SK6805-EC-15, F.Cu at (53.5, 130.0)
- added L8: SK6805-EC-15, progcc_v3:SK6805-EC-15, F.Cu at (48.6, 132.5)
- added R22: 330, Resistor_SMD:R_0402_1005Metric, F.Cu at (40.7, 136.5)
- added R23: 0, Resistor_SMD:R_0603_1608Metric_Pad0.98x0.95mm_HandSolder, F.Cu at (44.8, 129.7)
- added R24: 0, Resistor_SMD:R_0603_1608Metric_Pad0.98x0.95mm_HandSolder, F.Cu at (49.1, 129.7)
- added T1: 36-8730, progcc_v3:KS_8730, F.Cu at (48.3, 157.5)
- added T2: 36-8730, progcc_v3:KS_8730, F.Cu at (22.9, 157.5)
- added T3: 36-8730, progcc_v3:KS_8730, F.Cu at (30.5, 157.5)
- added T4: 36-8730, progcc_v3:KS_8730, F.Cu at (38.4, 157.5)
- added TP1: TestPoint, TestPoint:TestPoint_Pad_D1.5mm, F.Cu at (60.4, 130.2)
- added TP10: TestPoint, TestPoint:TestPoint_Pad_D1.5mm, F.Cu at (48.4, 140.3)
- added TP11: TestPoint, TestPoint:TestPoint_Pad_D1.5mm, F.Cu at (55.5, 134.0)
- added TP12: TestPoint, TestPoint:TestPoint_Pad_D1.5mm, F.Cu at (56.9, 130.2)
- added TP13: TestPoint, TestPoint:TestPoint_Pad_D1.5mm, F.Cu at (43.5, 144.1)
- added TP14: TestPoint, TestPoint:TestPoint_Pad_D1.5mm, F.Cu at (52.0, 134.0)
- added TP2: TestPoint, TestPoint:TestPoint_Pad_D1.5mm, F.Cu at (52.0, 137.6)
- added TP3: TestPoint, TestPoint:TestPoint_Pad_D1.5mm, F.Cu at (51.9, 141.1)
- added TP4: TestPoint, TestPoint:TestPoint_Pad_D1.5mm, F.Cu at (55.9, 147.4)
- added TP5: TestPoint, TestPoint:TestPoint_Pad_D1.5mm, F.Cu at (47.1, 143.9)
- added TP6: TestPoint, TestPoint:TestPoint_Pad_D1.5mm, F.Cu at (55.5, 137.6)
- added TP7: TestPoint, TestPoint:TestPoint_Pad_D1.5mm, F.Cu at (59.1, 133.8)
- added TP8: TestPoint, TestPoint:TestPoint_Pad_D1.5mm, F.Cu at (64.0, 130.2)
- added TP9: TestPoint, TestPoint:TestPoint_Pad_D1.5mm, F.Cu at (44.8, 140.3)
- added U10: MCP3002, progcc_v3:SOIC-8_3.9x4.9mm_P1.27mm, F.Cu at (33.2, 131.7)
- C10, C11, C9: value 100n -> .047u; footprint Capacitor_SMD:C_0402_1005Metric -> Capacitor_SMD:C_0603_1608Metric_Pad1.08x0.95mm_HandSolder
- C13: value 1u -> 100n
- C14: value .047u -> 100n; footprint Capacitor_SMD:C_0603_1608Metric_Pad1.08x0.95mm_HandSolder -> Capacitor_SMD:C_0402_1005Metric
- C15: value .047u -> 1u; footprint Capacitor_SMD:C_0603_1608Metric_Pad1.08x0.95mm_HandSolder -> Capacitor_SMD:C_0402_1005Metric
- C16, C17, C18: value 1u -> 100n; footprint Capacitor_SMD:C_0603_1608Metric -> Capacitor_SMD:C_0402_1005Metric
- C19: footprint Capacitor_SMD:C_0603_1608Metric -> Capacitor_SMD:C_0402_1005Metric
- C2: value 1u -> 2.2uF; footprint Capacitor_SMD:C_0402_1005Metric -> Capacitor_SMD:C_0603_1608Metric
- C22: value 10u -> 100n; footprint Capacitor_SMD:C_0603_1608Metric -> Capacitor_SMD:C_0402_1005Metric
- C3: value 6.3V 47uF -> 47uF 6.3v
- C4: value 10u -> 2.2uF
- C8: value .047u -> 10u; footprint Capacitor_SMD:C_0603_1608Metric_Pad1.08x0.95mm_HandSolder -> Capacitor_SMD:C_0603_1608Metric
- SW3: value TS09-63-25-R-260-SMT -> TS-1187A-B-A-B; footprint progcc_v3:TS09 -> progcc_v3:SW_TS-1187A-B-A-B
- U7: value MCP3002 -> LP3986-33B3F; footprint progcc_v3:SOIC-8_3.9x4.9mm_P1.27mm -> Package_TO_SOT_SMD:SOT-23
- moved C12 30.1 mm to (91.4, 99.1)
- moved U7 16.1 mm to (134.6, 111.8)
- moved J4 11.6 mm to (111.8, 97.4), turned to 180 degrees
Connections:
- net /C_x_filt renamed P_LX
- net /C_y_filt renamed P_LY
- net GULI_CLK renamed GULI_DZONE
- C10 pad 1: +3V3 -> GND
- C10 pad 2: GND -> LX
- C11 pad 1: +3V3 -> GND
- C11 pad 2: GND -> LY
- C12 pad 2: LY -> RX
- C13 pad 1: +3V3 -> GND
- C13 pad 2: GND -> +1V1
- C14 pad 2: RX -> +1V1
- C15 pad 2: RY -> +1V1
- C16 pad 1: +3.3V -> +3V3
- C17 pad 1: +3.3V -> +3V3
- C18 pad 1: +3.3V -> +3V3
- C19 pad 1: +3.3V -> +3V3
- C2 pad 1: GND -> +5V
- C2 pad 2: +1V1 -> GND
- C22 pad 1: +5V -> GND
- C22 pad 2: GND -> +3V3
- C3 pad 1: GND -> Net-(C3-Pad1)
- C3 pad 2: Net-(C3-Pad2) -> GND
- C4 pad 1: +3V3 -> Net-(C4-Pad1)
- C8 pad 2: LX -> +3V3
- C9 pad 1: +3V3 -> GND
- C9 pad 2: GND -> RY
- D2 pad 2: Net-(C3-Pad2) -> Net-(C3-Pad1)
- D3 pad 2: Net-(D3-Pad2) -> Net-(C4-Pad1)
- F2 pad 2: Net-(C3-Pad2) -> Net-(C3-Pad1)
- J3 pad 3: LED_EN -> BUTTON_RGB
- J9 pad S1: unconnected-(J9-PadS1) -> GND
- JP1 pad 1: GULI_DAT -> GULI_CALIBRATE
- SW1 pad S2: GND -> LS_BUTTON
- SW1 pad S3: LS_BUTTON -> GND
- SW2 pad S2: GND -> RS_BUTTON
- SW2 pad S3: RS_BUTTON -> GND
- U5 pad 2: GULI_DAT -> GULI_CALIBRATE
- U6 pad 11: unconnected-(U6-Pad11) -> N_CLOCK_3.3
- U6 pad 12: unconnected-(U6-Pad12) -> N_LATCH_3.3
- U6 pad 15: /GPIO12 -> unconnected-(U6-Pad15)
- U6 pad 16: Push_A -> unconnected-(U6-Pad16)
- U6 pad 17: /GPIO14 -> unconnected-(U6-Pad17)
- U6 pad 18: /GPIO15 -> RGB_OUT
- U6 pad 19: unconnected-(U6-Pad19) -> GND
- U6 pad 2: unconnected-(U6-Pad2) -> P_TX
- U6 pad 27: Scan_C -> Push_A
- U6 pad 28: Push_B -> Scan_C
- U6 pad 29: Scan_D -> Push_B
- U6 pad 3: unconnected-(U6-Pad3) -> GPIO1
- U6 pad 30: Scan_B -> Scan_D
- U6 pad 31: Push_C -> Scan_B
- U6 pad 32: Push_D -> Push_C
- U6 pad 34: Scan_A -> Push_D
- U6 pad 35: /CS2 -> Scan_A
- U6 pad 36: /CS1 -> R_BRAKE
- U6 pad 4: unconnected-(U6-Pad4) -> P_CLK
- U6 pad 40: N_DATA_3.3 -> unconnected-(U6-Pad40)
- U6 pad 41: R_BRAKE -> unconnected-(U6-Pad41)
- U6 pad 5: unconnected-(U6-Pad5) -> P_RX
- U6 pad 6: /Dout -> P_RCS
- U6 pad 7: unconnected-(U6-Pad7) -> GULI_CALIBRATE
- U6 pad 8: /CLK -> unconnected-(U6-Pad8)
- U6 pad 9: unconnected-(U6-Pad9) -> N_DATA_3.3
- U7 pad 1: /CS1 -> GND
- U7 pad 2: /Stick_x_filt -> Net-(C4-Pad1)
- U7 pad 3: /Stick_y_filt -> +5V
- U8 pad 1: /CS2 -> P_LCS
- U8 pad 5: /Din -> P_RX
- U8 pad 6: /Dout -> P_TX
- U8 pad 7: /CLK -> P_CLK
- U8 pad 8: VCC -> +3V3
Routing:
- net +1V1: track 18.6 -> 66.0 mm
- net LED_EN: track 36.1 -> 0.00 mm
- net BUTTON_RGB: track 0.00 -> 36.1 mm
- net LX: track 30.0 -> 0.00 mm
- net RY: track 26.0 -> 0.00 mm
- net +3V3: track 27.9 -> 52.1 mm
- net /QSPI_SD3: track 21.4 -> 0.00 mm
- net LY: track 12.1 -> 0.20 mm
- net +3.3V: track 21.2 -> 10.5 mm, vias 4 -> 2
- net Net-(C3-Pad2): track 6.18 -> 0.00 mm
- net Net-(C3-Pad1): track 0.00 -> 6.18 mm
- net Net-(C4-Pad1): track 0.00 -> 5.26 mm, vias 0 -> 1
- net Net-(F1-Pad2): track 0.13 -> 2.87 mm
- net GND: track 13.3 -> 15.9 mm, vias 2 -> 4
- net Net-(D3-Pad2): track 2.06 -> 0.00 mm
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
Commit message: More schematic fixes
Added some more schematic items, grouped RP2040 with caps on PCB.
Parts:
- moved T4 145.3 mm to (183.2, 145.4)
- moved T1 131.0 mm to (178.7, 145.4)
- moved L8 119.1 mm to (167.7, 131.9)
- moved L7 114.6 mm to (166.7, 148.6)
- moved L5 113.8 mm to (149.7, 133.8)
- moved C20 110.7 mm to (142.7, 119.7), turned to 180 degrees
- moved L6 108.7 mm to (150.0, 146.1)
- moved C23 106.8 mm to (142.7, 113.8), turned to 180 degrees
- moved C21 105.2 mm to (139.8, 119.2), turned to 90 degrees
- moved U10 104.4 mm to (137.4, 137.8), turned to 180 degrees
- moved U5 99.3 mm to (121.3, 134.6)
- moved C1 99.2 mm to (244.3, 145.9)
- moved C10 99.2 mm to (224.9, 159.4)
- moved C4 99.2 mm to (234.6, 142.7)
- moved D1 99.2 mm to (208.3, 147.5)
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Connections:
- L2 pad 1: SR_RGB -> Net-(L1-Pad3)
- L3 pad 1: Net-(L1-Pad3) -> Net-(L2-Pad3)
- L3 pad 3: Net-(L3-Pad3) -> Net-(L4-Pad1)
- L4 pad 1: Net-(L2-Pad3) -> Net-(L4-Pad1)
- L4 pad 3: Net-(L4-Pad3) -> SR_RGB
- L5 pad 1: Net-(L3-Pad3) -> SR_RGB
- L6 pad 1: Net-(L4-Pad3) -> Net-(L5-Pad3)
- L7 pad 1: Net-(L5-Pad3) -> Net-(L6-Pad3)
- L7 pad 3: SR_RGB -> Net-(L7-Pad3)
- L8 pad 1: Net-(L6-Pad3) -> Net-(L7-Pad3)
- U6 pad 8: unconnected-(U6-Pad8) -> GULI_DZONE
Routing:
- net +5V: track 77.8 -> 0.00 mm, vias 3 -> 0
- net +1V1: track 66.0 -> 12.5 mm, vias 3 -> 0
- net Scan_C: track 44.0 -> 0.00 mm
- net Scan_D: track 43.1 -> 0.00 mm
- net Push_B: track 42.6 -> 0.00 mm
- net Scan_B: track 42.4 -> 0.00 mm
- net Push_C: track 41.5 -> 0.00 mm
- net Push_D: track 40.6 -> 0.00 mm
- net Scan_A: track 40.2 -> 0.00 mm
- net RUMBLE-: track 39.3 -> 0.00 mm
- net Push_A: track 37.3 -> 0.00 mm
- net BUTTON_RGB: track 36.1 -> 0.00 mm
- net RX: track 33.6 -> 0.00 mm
- net +3V3: track 52.1 -> 20.4 mm, vias 9 -> 0
- net /~{USB_BOOT}: track 19.4 -> 0.00 mm, vias 2 -> 0
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- removed copper zone on In1.Cu, net +3V3
- removed copper zone on B.Cu, net GND
- removed copper zone on F.Cu, net GND
- removed copper zone on In2.Cu, net GND
Other:
- board text added: "ProGCC V3"
- board text removed: "Thingama Pro 2.1"

Commit message: some positioning changes+fP adjustments
Parts:
- added J1: Rumble, progcc_v3:rumble_pins, F.Cu at (179.8, 142.8)
- added J2: Rumble, progcc_v3:rumble_pins, F.Cu at (93.7, 138.7)
- C5, C6, C7: footprint Capacitor_SMD:C_0603_1608Metric_Pad1.08x0.95mm_HandSolder -> Capacitor_SMD:C_0402_1005Metric
- JP1, JP2: footprint Jumper:SolderJumper-2_P1.3mm_Open_RoundedPad1.0x1.5mm -> Jumper:SolderJumper-2_P1.3mm_Open_TrianglePad1.0x1.5mm
- R20, R23, R24: footprint Resistor_SMD:R_0603_1608Metric_Pad0.98x0.95mm_HandSolder -> Resistor_SMD:R_0402_1005Metric
- moved SW3 140.3 mm to (126.6, 96.9)
- moved C11 132.3 mm to (108.4, 119.1), turned to 180 degrees
- moved C10 130.9 mm to (97.4, 129.9), turned to -90 degrees
- moved TP9 127.7 mm to (163.0, 91.8)
- moved C15 122.3 mm to (22.4, 118.5), turned to 0 degrees
- moved C23 120.7 mm to (22.4, 123.0)
- moved C20 120.4 mm to (22.3, 120.8)
- moved TP14 115.5 mm to (159.5, 91.8)
- moved C16 113.6 mm to (22.3, 121.9), turned to 0 degrees
- moved C2 109.4 mm to (137.8, 110.8), turned to 0 degrees
- moved C14 108.2 mm to (22.4, 119.5)
- moved C4 103.6 mm to (137.8, 105.8), turned to 180 degrees
- moved F2 102.6 mm to (118.2, 119.2), turned to 90 degrees
- moved C3 100.8 mm to (120.7, 119.3), turned to 90 degrees
- moved R9 99.4 mm to (131.1, 99.8)
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Connections:
- J9 pad S1: GND -> unconnected-(J9-PadS1)
- U10 pad 2: P_RX -> RX
- U10 pad 3: P_RY -> RY
- U5 pad 6: G_LY -> LY
- U5 pad 7: G_LX -> LX
- U5 pad 8: G_RY -> RY
- U5 pad 9: G_RX -> RX
- U8 pad 2: P_LX -> LX
- U8 pad 3: P_LY -> LY
Routing:
- net +3.3V_PRE: track 0.00 -> 21.4 mm, vias 0 -> 1
- net +5V_PRE: track 0.00 -> 10.4 mm
- net /CC2: track 0.00 -> 10.0 mm
- net +1V1: track 12.5 -> 2.79 mm
- net N_LATCH: track 0.00 -> 8.35 mm, vias 0 -> 2
- net /CC1: track 0.00 -> 8.09 mm, vias 0 -> 2
- net N_DATA: track 0.00 -> 7.26 mm, vias 0 -> 1
- net +3V3: track 20.4 -> 13.2 mm, vias 0 -> 2
- net Net-(C3-Pad1): track 0.00 -> 7.06 mm
- net N_CLOCK: track 0.00 -> 6.06 mm, vias 0 -> 2
- net D-: track 0.00 -> 4.66 mm, vias 0 -> 1
- net D+: track 0.00 -> 4.22 mm, vias 0 -> 1
- net GND: track 0.00 -> 2.46 mm, vias 0 -> 1
- net /QSPI_SD3: track 0.00 -> 2.39 mm
- net RUMBLE-: track 0.00 -> 2.37 mm
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- added copper zone on In1.Cu, net +3V3
- added copper zone on B.Cu, net GND
- added copper zone on F.Cu, net GND
- added copper zone on In2.Cu, net GND

Commit message: USB C routing area
Parts:
- moved R9 16.8 mm to (147.6, 102.5), turned to 0 degrees
- moved SW3 13.8 mm to (112.9, 95.3)
- moved R8 2.19 mm to (147.6, 104.2)
Routing:
- net N_CLOCK: track 6.06 -> 16.3 mm
- net N_LATCH: track 8.35 -> 16.3 mm
- net N_DATA: track 7.26 -> 14.3 mm, vias 1 -> 2
- net /CC2: track 10.0 -> 16.9 mm, vias 0 -> 1
- net +5V_PRE: track 10.4 -> 16.0 mm, vias 0 -> 1
- net /CC1: track 8.09 -> 12.7 mm, vias 2 -> 1
- net +3.3V_PRE: track 21.4 -> 18.2 mm, vias 1 -> 2
- net D-: track 4.66 -> 7.61 mm, vias 1 -> 2
- net GND: track 2.46 -> 0.00 mm, vias 1 -> 0
- net D+: track 4.22 -> 6.15 mm

Commit message: major routing
most of the board is routed minus a couple bits
Parts:
- TP1, TP10, TP11, TP12, TP13, TP14, TP2, TP3, TP4, TP5, TP7, TP8, TP9: footprint TestPoint:TestPoint_Pad_D1.5mm -> progcc_v3:TestPoint_Pad_D1mm
- TP6: footprint TestPoint:TestPoint_Pad_D1.5mm -> Heatsink:TestPoint_Pad_D1mm
- moved TP4 87.7 mm to (131.8, 103.5)
- moved TP7 85.1 mm to (126.1, 105.3)
- moved TP5 84.8 mm to (125.9, 112.7)
- moved TP6 83.1 mm to (125.9, 108.9)
- moved TP3 79.1 mm to (119.4, 107.8)
- moved TP1 79.0 mm to (119.4, 114.7)
- moved TP2 73.5 mm to (119.4, 111.3)
- moved R13 59.6 mm to (128.1, 106.9)
- moved Q6 59.6 mm to (124.0, 106.8)
- moved R10 59.6 mm to (120.9, 106.9)
- moved R11 59.5 mm to (128.1, 113.9)
- moved Q5 59.4 mm to (124.0, 110.4)
- moved R12 59.4 mm to (128.1, 110.4)
- moved Q4 59.3 mm to (124.0, 113.9)
- moved R7 59.2 mm to (120.9, 110.4)
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Connections:
- C6 pad 1: +3.3V -> +3V3
- C7 pad 1: +3.3V -> +3V3
- Q4 pad 1: +3.3V -> +3V3
- Q5 pad 1: +3.3V -> +3V3
- Q6 pad 1: +3.3V -> +3V3
- R10 pad 1: +3.3V -> +3V3
- R20 pad 1: +3.3V -> +3V3
- R6 pad 1: +3.3V -> +3V3
- R7 pad 1: +3.3V -> +3V3
- U1 pad 1: +3.3V -> +3V3
- U2 pad 1: +3.3V -> +3V3
- U3 pad 1: +3.3V -> +3V3
- U4 pad 1: +3.3V -> +3V3
- U5 pad 1: +3.3V -> +3V3
Routing:
- net +5V: track 1.03 -> 72.2 mm, vias 0 -> 2
- net RX: track 0.00 -> 55.8 mm, vias 0 -> 4
- net P_TX: track 0.00 -> 53.8 mm, vias 0 -> 3
- net P_CLK: track 0.00 -> 53.2 mm, vias 0 -> 3
- net RY: track 0.00 -> 51.7 mm
- net +3V3: track 13.2 -> 63.6 mm, vias 2 -> 30
- net Push_D: track 0.00 -> 47.9 mm
- net Scan_A: track 0.00 -> 47.9 mm
- net Scan_D: track 0.00 -> 47.3 mm
- net Scan_B: track 0.00 -> 47.3 mm
- net Push_A: track 0.00 -> 47.2 mm
- net Push_C: track 0.00 -> 47.2 mm
- net Push_B: track 0.00 -> 47.2 mm
- net Scan_C: track 0.00 -> 46.5 mm
- net P_RX: track 0.00 -> 46.2 mm, vias 0 -> 3
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