File: progcc_v3_main/procon_gcc_main_pcb.kicad_sch (KiCad schematic)
At the start: 81 parts, among them J1 Rumble, J3 To Button Board, J4 Conn_01x06_Female, J5 Conn_01x02, J6 Conn_01x03_Male, J7 Rumble, J9 USB_C_Receptacle, Q1 Q_PMOS_GDS, Q2 Q_NMOS_GSD, Q3 Q_NMOS_GSD, SW1 SW_DIP_x04, SW3 SW_DIP_x01, U10 DRV5055A2xDBZxQ1, U11 DRV5055A2xDBZxQ1, U12 MCP3002, U13 PRTR5V0U2X, U14 XC6206PxxxMR, U15 RP2040, U2 2x DRV5053CAQLPGM Hall Effect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, U3 Stickbox_Assembly, U6 MCP3002, U7 DRV5055A2xDBZxQ1, U8 DRV5055A2xDBZxQ1, U9 W25Q128JVS, Y1 Crystal_GND3

Commit message: Update naming schema
Other:
- company: Luberry's Custom Controllers -> HHL/Esca
- title: Procon GCC Main PCB -> ProGCC v3 Main Board
Changed lines of the file:
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@@
   (paper "B")
   (title_block
-    (title "Procon GCC Main PCB")
+    (title "ProGCC v3 Main Board")
     (date "2019-12-18")
     (rev "0.1")
-    (company "Luberry's Custom Controllers")
+    (company "HHL/Esca")
   )
   (junction (at 307.975 64.135) (diameter 0) (color 0 0 0 0)

Commit message: Lots of schematic changes and upgrades
Good luck :P
Parts:
- removed C16, C17, C18: 0.047u, PhobGCC_Footprints:C_0603_HandSoldering, symbol Device:C
- removed C19, C20: 0.047u, Capacitor_SMD:C_0402_1005Metric, symbol Device:C
- removed C21, C31, C32, C33: 1u, PhobGCC_Footprints:C_0603_1608Metric_Pad1.08x0.95mm_HandSolder, symbol Device:C
- removed C23: 10u, Capacitor_SMD:C_0603_1608Metric, symbol Device:C
- removed D2, D8: MBR0520, Diode_SMD:D_SOD-323, symbol Diode:MBR0520
- removed D4, D5, D6, D7: D_Small, Diode_SMD:D_SOD-123, symbol Device:D_Small
- removed J5: Conn_01x02, PhobGCC_2_0_0_footprints:PinHeader_1x02_P2.00mm_Vertical, symbol Connector_Generic:Conn_01x02
- removed Q2, Q3: Q_NMOS_GSD, PhobGCC_Footprints:SOT-23, symbol Device:Q_NMOS_GSD
- removed R22, R24, R26, R28: 316, Resistor_SMD:R_0603_1608Metric, symbol Device:R
- removed R23, R25, R27: 180, Resistor_SMD:R_0603_1608Metric, symbol Device:R
- removed S1: BOOTSEL, PhobGCC_2_0_0_footprints:SW_TS-1187A-B-A-B, symbol TS-1187A-B-A-B:TS-1187A-B-A-B
- removed SW1: SW_DIP_x04, dips:C54962_4pos, symbol Switch:SW_DIP_x04
- removed SW3: SW_DIP_x01, dips:switch_C381098, symbol Switch:SW_DIP_x01
- removed U10, U11, U7, U8: DRV5055A2xDBZxQ1, PhobGCC_2_0_0_footprints:SOT-23, symbol Sensor_Magnetic:DRV5055A2xDBZxQ1
- removed U12, U6: MCP3002, PhobGCC_2_0_0_footprints:SOIC-8_3.9x4.9mm_P1.27mm, symbol Analog_ADC:MCP3002
- removed U13: PRTR5V0U2X, random-keyboard-parts:SOT143B, symbol cipulot_parts:PRTR5V0U2X
- removed U15: RP2040, PhobGCC_2_0_0_footprints:RP2040-QFN-56, symbol MCU_RaspberryPi_RP2040:RP2040
- removed U2: 2x DRV5053CAQLPGM Hall Effect Sensors, PhobGCC_Footprints:GCC_Stickbox_2, symbol GCC:Gamecube-MB-rescue_Stickbox_Assembly-Gamecube_MB
- removed U3: Stickbox_Assembly, PhobGCC_Footprints:GCC_Stickbox_Hall_Only, symbol Gamecube MB:Stickbox_Assembly_Hall_Only
- added C12, C14, C8: 1u, Capacitor_SMD:C_0603_1608Metric_Pad1.08x0.95mm_HandSolder, symbol Device:C
- added C4: 10u, Capacitor_SMD:C_0603_1608Metric, symbol Device:C
- added C5, C6: 4.7uF, Capacitor_SMD:C_0603_1608Metric_Pad1.08x0.95mm_HandSolder, symbol Device:C
- added C7: 0.1uF, Capacitor_SMD:C_0603_1608Metric_Pad1.08x0.95mm_HandSolder, symbol Device:C
- added D2, D3, D4: CUS08F30, Diode_SMD:D_SOD-323_HandSoldering, symbol progcc_v3:CUS08F30
- added F2, F3: Fuse, Fuse:Fuse_1206_3216Metric_Pad1.42x1.75mm_HandSolder, symbol Device:Fuse
- added JP1, JP2: SolderJumper_2_Open, Jumper:SolderJumper-2_P1.3mm_Open_RoundedPad1.0x1.5mm, symbol Jumper:SolderJumper_2_Open
- added Q2, Q3: Q_PMOS_GDS, Package_TO_SOT_SMD:SOT-23, symbol Device:Q_PMOS_GSD
- added Q4, Q5, Q6: BSS138, Package_TO_SOT_SMD:SOT-23, symbol Transistor_FET:BSS138
- added R10, R11: 1k, Resistor_SMD:R_0603_1608Metric_Pad0.98x0.95mm_HandSolder, symbol Device:R
- added SW1, SW2: GL18_SW, progcc_v3:GL18, symbol progcc_v3:GL18_SW
- added SW3: TS09-63-25-R-260-SMT, progcc_v3:TS09, symbol progcc_v3:TS09-63-25-R-260-SMT
- added U1, U2, U3, U4: GH39F (Hall SOT23), progcc_v3:GH39F, symbol progcc_v3:GH39F (Hall SOT23)
- added U5: GL16112, progcc_v3:MSOP10, symbol progcc_v3:GL16112
- added U6: RP2040, Package_DFN_QFN:QFN-56-1EP_7x7mm_P0.4mm_EP3.2x3.2mm, symbol progcc_v3:RP2040
- C15: value 0.047u -> 1u; footprint PhobGCC_Footprints:C_0603_HandSoldering -> Capacitor_SMD:C_0603_1608Metric_Pad1.08x0.95mm_HandSolder; LCSC C1622 -> C15849
- D1: footprint PhobGCC_Footprints:D_SOD-123 -> Diode_SMD:D_SOD-123; MPN (none) -> B5819W SL
- F1: footprint PhobGCC_Footprints:Fuse_1206_3216Metric -> Fuse:Fuse_1206_3216Metric_Pad1.42x1.75mm_HandSolder
- J1, J7: footprint PhobGCC_Footprints:rumble_pins -> Connector_PinHeader_2.00mm:PinHeader_1x02_P2.00mm_Horizontal
- J4: footprint PhobGCC_Footprints:GCC_Header_Straight_1x06_Pitch2.00mm -> Connector_PinHeader_2.00mm:PinHeader_1x06_P2.00mm_Horizontal
- J6: footprint PhobGCC_Footprints:PinHeader_1x01_P2.54mm_Vertical -> Connector_PinHeader_2.00mm:PinHeader_1x03_P2.00mm_Horizontal
- Q1: footprint PhobGCC_Footprints:SOT-23 -> Package_TO_SOT_SMD:SOT-23
- R1, R2, R3, R4, R5: footprint PhobGCC_Footprints:R_0603_1608Metric_Pad0.98x0.95mm_HandSolder -> Resistor_SMD:R_0603_1608Metric_Pad0.98x0.95mm_HandSolder
- R12, R13, R6, R7: value 10k -> 1k; footprint Resistor_SMD:R_0402_1005Metric -> Resistor_SMD:R_0603_1608Metric_Pad0.98x0.95mm_HandSolder
- R14: footprint PhobGCC_2_0_0_footprints:C_0402_1005Metric -> Resistor_SMD:R_0603_1608Metric_Pad0.98x0.95mm_HandSolder
- R15: value 2k -> 1k; footprint PhobGCC_Footprints:R_0603_1608Metric_Pad0.98x0.95mm_HandSolder -> Resistor_SMD:R_0603_1608Metric_Pad0.98x0.95mm_HandSolder; LCSC C22975 -> (none); Manufacturer PN 0603WAF1002T5ECopy -> (none)
- R16, R17, R18: value 2k -> 1k; footprint PhobGCC_Footprints:R_0603_1608Metric_Pad0.98x0.95mm_HandSolder -> Resistor_SMD:R_0603_1608Metric_Pad0.98x0.95mm_HandSolder; LCSC C22975 -> (none)
- R19, R29, R30: footprint Resistor_SMD:R_0402_1005Metric -> Resistor_SMD:R_0603_1608Metric_Pad0.98x0.95mm_HandSolder
- R20: value 180 -> 0; footprint Resistor_SMD:R_0603_1608Metric -> Resistor_SMD:R_0603_1608Metric_Pad0.98x0.95mm_HandSolder
- R21: value 180 -> 33; footprint Resistor_SMD:R_0603_1608Metric -> Resistor_SMD:R_0603_1608Metric_Pad0.98x0.95mm_HandSolder
- R8, R9: footprint PhobGCC_Footprints:R_0603_1608_DNP -> Resistor_SMD:R_0603_1608Metric_Pad0.98x0.95mm_HandSolder
- U9: footprint PhobGCC_2_0_0_footprints:SOIC-8_5.23x5.23mm_P1.27mm -> Package_SO:SOIC-8_5.23x5.23mm_P1.27mm
Connections:
- net +1V1: now also U6.23 (DVDD), U6.45 (VREG_VOUT), U6.50 (DVDD)
- net +3.3V: now also C15.1, R20.1, R6.1, R7.1, C12.1, C14.1, C6.1, C7.1, C8.1, Q4.1 (G), Q5.1 (G), Q6.1 (G), R10.1, U1.1 (VDD), U2.1 (VDD), U3.1 (VDD), U4.1 (VDD), U5.1 (VDD); no longer C3.2, J4.1 (Pin_1), J9.A2 (TX1+), J9.B2 (TX2+)
- net +3V3: now also C4.1, D2.1 (K), D3.1 (K), D4.2 (A), U6.1 (IOVDD), U6.10 (IOVDD), U6.22 (IOVDD), U6.33 (IOVDD), U6.42 (IOVDD), U6.43 (ADC_AVDD), U6.44 (VREG_IN), U6.48 (USB_VDD), U6.49 (IOVDD); no longer R12.1, R6.1
- net +5V: now also F3.2; no longer J4.2 (Pin_2), J9.A4 (VBUS), J9.A9 (VBUS), J9.B4 (VBUS), J9.B9 (VBUS)
- net CLK: now also U6.8 (GPIO6)
- net CS1: now also U6.36 (GPIO24)
- net CS2: now also U6.35 (GPIO23)
- net Dout: now also U6.6 (GPIO4)
- net GND: now also J9.S1 (SHIELD), C12.2, C14.2, C4.2, C5.2, C6.2, C7.2, C8.2, JP1.2 (B), JP2.2 (B), Q2.3 (D), Q3.3 (D), SW1.S3 (3), SW1.S4 (4), SW2.S3 (3), SW2.S4 (4), SW3.1, U1.3 (GND), U2.3 (GND), U3.3 (GND), U4.3 (GND), U5.10 (GND), U6.57 (GND); no longer R13.2, R20.2, R7.2
- net GPIO12: now also U6.15 (GPIO12)
- net GPIO14: now also U6.17 (GPIO14)
- net GPIO15: now also U6.18 (GPIO15)
- net Push_A: now also U6.16 (GPIO13)
- net Push_B: now also U6.28 (GPIO17)
- net Push_C: now also U6.31 (GPIO20)
- net Push_D: now also U6.32 (GPIO21)
- net QSPI_SCLK: now also U6.52 (QSPI_SCLK)
- net QSPI_SD0: now also U6.53 (QSPI_SD0)
- net QSPI_SD1: now also U6.55 (QSPI_SD1)
- net QSPI_SD2: now also U6.54 (QSPI_SD2)
- net QSPI_SD3: now also U6.51 (QSPI_SD3)
- net QSPI_SS: now also U6.56 (QSPI_SS)
- net RUN: now also U6.26 (RUN)
- net SWCLK: now also U6.24 (SWCLK)
- net SWD: now also U6.25 (SWD)
- net Scan_A: now also U6.34 (GPIO22)
- net Scan_B: now also U6.30 (GPIO19)
- net Scan_C: now also U6.27 (GPIO16)
- net Scan_D: now also U6.29 (GPIO18)
- net XTAL_IN: now also U6.20 (XIN)
- net XTAL_OUT: now also U6.21 (XOUT)
- net ~{USB_BOOT}: now also SW3.2
- net at Q1.1 (G), R1.1: now also Q2.2 (S)
- net RUMBLE-: now reaches D1.2 (A), F1.1, J1.2 (Pin_2), J7.2 (Pin_2), Q1.3 (D)
- net at R4.2: now also Q3.1 (G)
- net at F1.2: now also Q3.2 (S)
- net GULI_TXD: now reaches R21.1
- net at R29.2: now also U6.47 (USB_DP)
- net CC2: now reaches J9.B5 (CC2), R9.1
- net CC1: now reaches J9.A5 (CC1), R8.1
- net at R2.2: now also Q2.1 (G)
- net at R30.2: now also U6.46 (USB_DM)
- net at R21.2: now also U5.5 (PC3); no longer R20.1
- net N_LATCH: now reaches J9.A10 (RX2-)
- net N_LATCH: now also J9.B10 (RX1-), Q4.3 (D), R11.2
- net N_CLOCK: now reaches J9.A3 (TX1-)
- net N_CLOCK: now also J9.B3 (TX2-), R12.2, Q5.3 (D)
- net at U14.2 (VO): now also D3.2 (A)
- net ADC_Lx renamed LX
- net ADC_Ly renamed LY
- net ADC_Rx renamed RX
- net ADC_Ry renamed RY
- net Brake renamed R_BRAKE
- net R_BRAKE: now also U6.41 (GPIO29_ADC3)
- net C_x_filt: no longer names the net of R17.1
- net C_x_filt: now also U3.2 (VOUT)
- net C_y_filt: no longer names the net of R18.1
- net C_y_filt: now also U4.2 (VOUT)
- net Data renamed N_DATA
- net N_DATA: now also R13.2, Q6.3 (D)
- net Lanalog renamed N_LATCH_3.3
- net N_LATCH_3.3: now also Q4.2 (S); no longer R7.1
- net Ranalog renamed SHARED_PU
- net SHARED_PU: now also R12.1, D4.1 (K), R11.1; no longer R12.2
- net Rumble renamed RUMBLE
- net RUMBLE: now also U6.37 (GPIO25)
- net Stick_x_filt: no longer names the net of R15.1
- net Stick_x_filt: now also U1.2 (VOUT); no longer C15.1
- net Stick_y_filt: no longer names the net of R16.1
- net Stick_y_filt: now also U2.2 (VOUT)
- net d+ renamed D+
- net d- renamed D-
- new net: C3.2, D2.2 (A), F2.2
- new net: R20.2, U5.4 (PC2)
- new net +3.3V_PRE: F2.1, J4.1 (Pin_1), J9.A2 (TX1+), J9.B2 (TX2+)
- new net +5V_PRE: F3.1, J4.2 (Pin_2), J9.A4 (VBUS), J9.A9 (VBUS), J9.B4 (VBUS), J9.B9 (VBUS)
- new net GULI_CLK: JP2.1 (A), U5.3 (PC1(CLK))
- new net GULI_DAT: C5.1, JP1.1 (A), U5.2 (PC0(DAT))
- new net G_LX: U5.7 (AN2)
- new net G_LY: U5.6 (AN3)
- new net G_RX: U5.9 (AN0)
- new net G_RY: U5.8 (AN1)
- new net LS_BUTTON: SW1.S1 (1), SW1.S2 (2)
- new net N_CLOCK_3.3: Q5.2 (S), R7.2
- new net N_DATA_3.3: Q6.2 (S), R10.2, U6.40 (GPIO28_ADC2)
- new net RS_BUTTON: SW2.S1 (1), SW2.S2 (2)
Other:
- note added: "6 Pin GameCube Cable"
- note added: "GL Calibrate Enable"
- note added: "GL Deadzone Enable"
- note added: "Level Shifters"
- note removed: "6pin from gamecube"
- note removed: "Clock Gen"
- note removed: "Communication"
- note removed: "Data Connector"
- note removed: "Digital Trigger Conversion"
- note removed: "Joysticks"
- note removed: "Main ASIC"
- note removed: "Make sure C8 is close to pin 45 of RP2040"
- note removed: "Power"
- note removed: "Rumble load reduction"
- note removed: "Trigger Mode Selection"
- note removed: "Wired Data Connector"
- moved on the sheet: C1, C10, C11, C13, C2, C22, C9, D1, F1, J1, J3, J4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

Commit message: some schematic fixes+some positioning
Parts:
- removed J7: Rumble, Connector_PinHeader_2.00mm:PinHeader_1x02_P2.00mm_Horizontal, symbol Connector:Conn_01x02_Male
- added C16, C17, C18, C19: 1u, Capacitor_SMD:C_0603_1608Metric, symbol Device:C
- added J2: Rumble, progcc_v3:rumble_pins, symbol Connector:Conn_01x02_Male
- added U7, U8: MCP3002, progcc_v3:SOIC-8_3.9x4.9mm_P1.27mm, symbol Analog_ADC:MCP3002
- C12, C14, C15, C8: value 1u -> .047u
- J1: footprint Connector_PinHeader_2.00mm:PinHeader_1x02_P2.00mm_Horizontal -> progcc_v3:rumble_pins
- J4: footprint Connector_PinHeader_2.00mm:PinHeader_1x06_P2.00mm_Horizontal -> progcc_v3:GCC_Header_Straight_1x06_Pitch2.00mm
- J6: footprint Connector_PinHeader_2.00mm:PinHeader_1x03_P2.00mm_Horizontal -> progcc_v3:PinHeader_1x03_P2.54mm_Vertical
- R14, R19, R29, R30: footprint Resistor_SMD:R_0603_1608Metric_Pad0.98x0.95mm_HandSolder -> Resistor_SMD:R_0402_1005Metric
Connections:
- net +3.3V: now also C16.1, C17.1, C18.1, C19.1; no longer C12.1, C14.1, C15.1, C8.1
- net +3V3: now also U7.8 (VDD/VREF)
- net +5V: now also J2.1 (Pin_1)
- net CLK: now also U7.7 (CLK), U8.7 (CLK)
- net CS1: now also U7.1 (~{CS}/SHDN)
- net CS2: now also U8.1 (~{CS}/SHDN)
- net Dout: now also U7.6 (DOUT), U8.6 (DOUT)
- net GND: now also C12.1, C14.1, C15.1, C8.1, SW1.S2 (2), SW2.S2 (2), C16.2, C17.2, C18.2, C19.2, U7.4 (VSS), U8.4 (VSS); no longer C12.2, C14.2, C15.2, C8.2, J9.S1 (SHIELD), SW1.S3 (3), SW2.S3 (3)
- net LS_BUTTON: now also SW1.S3 (3); no longer SW1.S2 (2)
- net LX: now also C8.2
- net LY: now also C12.2
- net RS_BUTTON: now also SW2.S3 (3); no longer SW2.S2 (2)
- net RUMBLE-: now also J2.2 (Pin_2)
- net RX: now also C14.2
- net RY: now also C15.2
- new net C_x_filt: U8.2 (CH0)
- new net C_y_filt: U8.3 (CH1)
- new net Din: U7.5 (DIN), U8.5 (DIN)
- new net Stick_x_filt: U7.2 (CH0)
- new net Stick_y_filt: U7.3 (CH1)
- new net VCC: U8.8 (VDD/VREF)
Other:
- moved on the sheet: C12, C14, C15, C8

Commit message: Schematic finalization
Parts:
- removed C10: 100n, Capacitor_SMD:C_0402_1005Metric, symbol Device:C
- removed C19: 1u, Capacitor_SMD:C_0603_1608Metric, symbol Device:C
- removed C3: 6.3V 47uF, Capacitor_Tantalum_SMD:CP_EIA-3216-18_Kemet-A, symbol Device:C_Small
- removed J1, J2: Rumble, progcc_v3:rumble_pins, symbol Connector:Conn_01x02_Male
- removed J6: Conn_01x03_Male, progcc_v3:PinHeader_1x03_P2.54mm_Vertical, symbol Connector:Conn_01x03_Male
- removed SW3: TS09-63-25-R-260-SMT, progcc_v3:TS09, symbol progcc_v3:TS09-63-25-R-260-SMT
- removed U14: XC6206PxxxMR, Package_TO_SOT_SMD:SOT-23, symbol Regulator_Linear:XC6206PxxxMR
- added C13, C20, C21, C23: 100n, Capacitor_SMD:C_0402_1005Metric, symbol Device:C
- added C3: 47uF 6.3v, Capacitor_Tantalum_SMD:CP_EIA-3216-18_Kemet-A, symbol Device:C_Polarized
- added C8: 10u, Capacitor_SMD:C_0603_1608Metric, symbol Device:C
- added L1, L2, L3, L4, L5, L6, L7, L8: SK6805-EC-15, progcc_v3:SK6805-EC-15, symbol progcc_v3:SK6805-EC-15
- added R22: 330, Resistor_SMD:R_0402_1005Metric, symbol Device:R
- added R23, R24: 0, Resistor_SMD:R_0603_1608Metric_Pad0.98x0.95mm_HandSolder, symbol Device:R
- added SW3: TS-1187A-B-A-B, progcc_v3:SW_TS-1187A-B-A-B, symbol progcc_v3:TS-1187A-B-A-B
- added T1, T2, T3, T4: 36-8730, progcc_v3:KS_8730, symbol Connector:TestPoint
- added TP1, TP10, TP11, TP12, TP13, TP14, TP2, TP3, TP4, TP5, TP6, TP7, TP8, TP9: TestPoint, TestPoint:TestPoint_Pad_D1.5mm, symbol Connector:TestPoint
- added U7: LP3986-33B3F, Package_TO_SOT_SMD:SOT-23, symbol Regulator_Linear:AP2127N-3.3
- C11, C9: value 100n -> .047u; footprint Capacitor_SMD:C_0402_1005Metric -> Capacitor_SMD:C_0603_1608Metric_Pad1.08x0.95mm_HandSolder; LCSC (none) -> C15849
- C14: value .047u -> 100n; footprint Capacitor_SMD:C_0603_1608Metric_Pad1.08x0.95mm_HandSolder -> Capacitor_SMD:C_0402_1005Metric; LCSC C15849 -> (none)
- C15: value .047u -> 1u; footprint Capacitor_SMD:C_0603_1608Metric_Pad1.08x0.95mm_HandSolder -> Capacitor_SMD:C_0402_1005Metric; LCSC C15849 -> (none)
- C16, C17, C18: value 1u -> 100n; footprint Capacitor_SMD:C_0603_1608Metric -> Capacitor_SMD:C_0402_1005Metric; LCSC C15849 -> (none)
- C2: value 1u -> 2.2uF; footprint Capacitor_SMD:C_0402_1005Metric -> Capacitor_SMD:C_0603_1608Metric
- C22: value 10u -> 100n; footprint Capacitor_SMD:C_0603_1608Metric -> Capacitor_SMD:C_0402_1005Metric
- C4: value 10u -> 2.2uF
- renumbered C8 to C10, C13 to C19, U8 to U10, U7 to U8
Connections:
- net C_x_filt is gone; now on net P_RX: U10.2 (CH0)
- net Din is gone; now on net P_RX: U10.5 (DIN), U8.5 (DIN)
- net VCC is gone; now on net +3V3: U10.8 (VDD/VREF)
- net +1V1: now also C14.2, C15.2, C13.2; no longer C2.2
- net +3.3V: no longer C16.1, C17.1, C18.1
- net +3V3: now also C16.1, C17.1, C18.1, C22.2, C20.2, C21.2, C23.2, C8.2, L1.2 (VDD), L2.2 (VDD), L3.2 (VDD), L4.2 (VDD), L5.2 (VDD), L6.2 (VDD), L7.2 (VDD), L8.2 (VDD), TP14.1; no longer C11.1, C4.1, C9.1
- net +5V: now also C2.1, T1.1, T3.1, TP9.1, U7.3 (VI); no longer C22.1
- net GND: now also C11.1, C2.2, C22.1, C9.1, J9.S1 (SHIELD), SW1.S3 (3), SW2.S3 (3), U6.19 (TESTEN), C13.1, C20.1, C21.1, C23.1, C3.2, C8.1, L1.4 (GND), L2.4 (GND), L3.4 (GND), L4.4 (GND), L5.4 (GND), L6.4 (GND), L7.4 (GND), L8.4 (GND), SW3.A, SW3.B, U7.1 (GND); no longer C11.2, C2.1, C22.2, C9.2, SW1.S2 (2), SW2.S2 (2)
- net GULI_DAT: no longer JP1.1 (A), U5.2 (PC0(DAT))
- net GULI_TXD: now also R24.1
- net LS_BUTTON: now also SW1.S2 (2); no longer SW1.S3 (3)
- net LY: now also C11.2; no longer C12.2
- net N_CLOCK: now also TP6.1
- net N_CLOCK_3.3: now also U6.11 (GPIO8), TP2.1
- net N_DATA: now also TP7.1
- net N_DATA_3.3: now also U6.9 (GPIO7), TP3.1; no longer U6.40 (GPIO28_ADC2)
- net N_LATCH: now also TP5.1
- net N_LATCH_3.3: now also U6.12 (GPIO9), TP1.1
- net Push_A: now also U6.27 (GPIO16); no longer U6.16 (GPIO13)
- net Push_B: now also U6.29 (GPIO18); no longer U6.28 (GPIO17)
- net Push_C: now also U6.32 (GPIO21); no longer U6.31 (GPIO20)
- net Push_D: now also U6.34 (GPIO22); no longer U6.32 (GPIO21)
- net RS_BUTTON: now also SW2.S2 (2); no longer SW2.S3 (3)
- net RUMBLE: now also TP11.1
- net RUMBLE-: now also T2.1, T4.1
- net RX: now also C12.2; no longer C14.2
- net RY: now also C9.2; no longer C15.2
- net R_BRAKE: now also U6.36 (GPIO24), TP8.1; no longer U6.41 (GPIO29_ADC3)
- net SHARED_PU: now also TP4.1
- net Scan_A: now also U6.35 (GPIO23); no longer U6.34 (GPIO22)
- net Scan_B: now also U6.31 (GPIO20); no longer U6.30 (GPIO19)
- net Scan_C: now also U6.28 (GPIO17); no longer U6.27 (GPIO16)
- net Scan_D: now also U6.30 (GPIO19); no longer U6.29 (GPIO18)
- net ~{USB_BOOT}: now also SW3.C, SW3.D
- net at D3.2 (A): now also C4.1, TP13.1, U7.2 (VO)
- net at D2.2 (A), F2.2: now also C3.1, TP10.1, TP12.1
- net P_TX: now reaches U6.2 (GPIO0)
- net P_TX: now also U10.6 (DOUT), U8.6 (DOUT)
- net GPIO1: now reaches U6.3 (GPIO1)
- net GPIO1: now also R23.2, R24.2
- net P_CLK: now reaches U6.4 (GPIO2)
- net P_CLK: now also U10.7 (CLK), U8.7 (CLK)
- net P_RX: now reaches U6.5 (GPIO3)
- net GULI_CALIBRATE: now reaches U6.7 (GPIO5)
- net GULI_CALIBRATE: now also JP1.1 (A), U5.2 (PC0(DAT))
- removed net CLK: U10.7 (CLK), U6.8 (GPIO6), U8.7 (CLK)
- net CS1 renamed P_LCS
- net P_LCS: now also R23.1; no longer U6.36 (GPIO24)
- net CS2 renamed P_RCS
- net P_RCS: now also U6.6 (GPIO4); no longer U6.35 (GPIO23)
- net C_y_filt renamed P_RY
- removed net Dout: U10.6 (DOUT), U6.6 (GPIO4), U8.6 (DOUT)
- net GPIO12: no longer names the net of U6.15 (GPIO12)
- net GPIO14: no longer names the net of U6.17 (GPIO14)
- net GPIO15 renamed RGB_OUT
- net RGB_OUT: now also R22.2
- net GULI_CLK renamed GULI_DZONE
- net GULI_DZONE: now also U6.8 (GPIO6)
- net LED_EN renamed BUTTON_RGB
- net BUTTON_RGB: now also L8.3 (DOUT)
- net Stick_x_filt renamed P_LX
- net Stick_y_filt renamed P_LY
- new net: L2.3 (DOUT), L4.1 (DIN)
- new net: L4.3 (DOUT), L6.1 (DIN)
- new net: L6.3 (DOUT), L8.1 (DIN)
- new net: L3.3 (DOUT), L5.1 (DIN)
- new net: L5.3 (DOUT), L7.1 (DIN)
- new net: L1.3 (DOUT), L3.1 (DIN)
- new net SL_RGB: L1.1 (DIN), R22.1
- new net SR_RGB: L2.1 (DIN), L7.3 (DOUT)
Other:
- note added: "Alternate ADC Selection"
- note added: "Alternate ADCs"
- note added: "GuliKit ADC IC"
- note added: "GuliKit Sticks"
- note added: "Hall Sensors"
- note added: "Power Bus"
- note added: "RGB LEDs"
- note added: "RP2040"
- note added: "Rumble"
- note added: "Rumble Connection"
- moved on the sheet: C1, C10, C19, C5, C6, C7, D1, D2, D3, D4, F1, F2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
