File: progcc_v3_main/procon_gcc_main_pcb.kicad_sch (KiCad schematic)
At the start: 107 parts, among them J3 To Button Board, J4 Conn_01x06_Female, J9 USB_C_Receptacle, Q1 Q_PMOS_GDS, Q2 Q_PMOS_GDS, Q3 Q_PMOS_GDS, Q4 BSS138, Q5 BSS138, Q6 BSS138, SW1 GL18_SW, SW2 GL18_SW, SW3 TS-1187A-B-A-B, T1 36-8730, T2 36-8730, T3 36-8730, T4 36-8730, U1 GH39F (Hall SOT23), U10 MCP3002, U2 GH39F (Hall SOT23), U3 GH39F (Hall SOT23), U4 GH39F (Hall SOT23), U5 GL16112, U6 RP2040, U7 LP3986-33B3F, U8 MCP3002, U9 W25Q128JVS, Y1 Crystal_GND3

Commit message: More schematic fixes
Added some more schematic items, grouped RP2040 with caps on PCB.
Parts:
- renumbered L3 to L2, L5 to L3, L7 to L4, L2 to L5, L4 to L6, L6 to L7
Connections:
- net G_LX is gone; now on net LX: U5.7 (AN2)
- net G_LY is gone; now on net LY: U5.6 (AN3)
- net G_RX is gone; now on net RX: U5.9 (AN0)
- net G_RY is gone; now on net RY: U5.8 (AN1)
- net P_LX is gone; now on net LX: U8.2 (CH0)
- net P_LY is gone; now on net LY: U8.3 (CH1)
- net P_RY is gone; now on net RY: U10.3 (CH1)
- net P_RX: no longer U10.2 (CH0)
- net RX: now also U10.2 (CH0)
Changed lines of the file:
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@@
     )
   )
-  (global_label "G_RY" (shape input) (at 66.04 215.9 0) (fields_autoplaced)
+  (global_label "RY" (shape input) (at 66.04 215.9 0) (fields_autoplaced)
     (effects (font (size 1.27 1.27)) (justify left))
-    (property "Intersheet References" "${INTERSHEET_REFS}" (id 0) (at 72.9604 215.8206 0)
+    (property "Intersheet References" "${INTERSHEET_REFS}" (id 0) (at 70.7228 215.8206 0)
       (effects (font (size 1.27 1.27)) (justify left) hide)
     )
@@
     )
   )
-  (global_label "G_LY" (shape input) (at 66.04 220.98 0) (fields_autoplaced)
+  (global_label "LY" (shape input) (at 66.04 220.98 0) (fields_autoplaced)
     (effects (font (size 1.27 1.27)) (justify left))
-    (property "Intersheet References" "${INTERSHEET_REFS}" (id 0) (at 72.7185 220.9006 0)
+    (property "Intersheet References" "${INTERSHEET_REFS}" (id 0) (at 70.4809 220.9006 0)
       (effects (font (size 1.27 1.27)) (justify left) hide)
     )
@@
     )
   )
-  (global_label "P_RY" (shape input) (at 238.76 76.2 180) (fields_autoplaced)
+  (global_label "RY" (shape input) (at 238.76 76.2 180) (fields_autoplaced)
     (effects (font (size 1.27 1.27)) (justify right))
-    (property "Intersheet References" "${INTERSHEET_REFS}" (id 0) (at 231.8396 76.1206 0)
+    (property "Intersheet References" "${INTERSHEET_REFS}" (id 0) (at 234.0772 76.1206 0)
       (effects (font (size 1.27 1.27)) (justify right) hide)
     )
   )
-  (global_label "P_LX" (shape input) (at 237.49 33.02 180) (fields_autoplaced)
+  (global_label "LX" (shape input) (at 237.49 33.02 180) (fields_autoplaced)
     (effects (font (size 1.27 1.27)) (justify right))
-    (property "Intersheet References" "${INTERSHEET_REFS}" (id 0) (at 230.6906 32.9406 0)
+    (property "Intersheet References" "${INTERSHEET_REFS}" (id 0) (at 232.9282 32.9406 0)
       (effects (font (size 1.27 1.27)) (justify right) hide)
     )
@@
     )
   )
-  (global_label "G_RX" (shape input) (at 66.04 213.36 0) (fields_autoplaced)
+  (global_label "RX" (shape input) (at 66.04 213.36 0) (fields_autoplaced)
     (effects (font (size 1.27 1.27)) (justify left))
-    (property "Intersheet References" "${INTERSHEET_REFS}" (id 0) (at 73.0813 213.2806 0)
+    (property "Intersheet References" "${INTERSHEET_REFS}" (id 0) (at 70.8437 213.2806 0)
       (effects (font (size 1.27 1.27)) (justify left) hide)
     )
@@
     )
   )
-  (global_label "G_LX" (shape input) (at 66.04 218.44 0) (fields_autoplaced)
+  (global_label "LX" (shape input) (at 66.04 218.44 0) (fields_autoplaced)
     (effects (font (size 1.27 1.27)) (justify left))
-    (property "Intersheet References" "${INTERSHEET_REFS}" (id 0) (at 72.8394 218.3606 0)
+    (property "Intersheet References" "${INTERSHEET_REFS}" (id 0) (at 70.6018 218.3606 0)
       (effects (font (size 1.27 1.27)) (justify left) hide)
     )
@@
     )
   )
-  (global_label "P_RX" (shape input) (at 238.76 66.04 180) (fields_autoplaced)
+  (global_label "RX" (shape input) (at 238.76 66.04 180) (fields_autoplaced)
     (effects (font (size 1.27 1.27)) (justify right))
-    (property "Intersheet References" "${INTERSHEET_REFS}" (id 0) (at 231.7187 65.9606 0)
+    (property "Intersheet References" "${INTERSHEET_REFS}" (id 0) (at 233.9563 65.9606 0)
       (effects (font (size 1.27 1.27)) (justify right) hide)
     )
   )
-  (global_label "P_LY" (shape input) (at 237.49 43.18 180) (fields_autoplaced)
+  (global_label "LY" (shape input) (at 237.49 43.18 180) (fields_autoplaced)
     (effects (font (size 1.27 1.27)) (justify right))
-    (property "Intersheet References" "${INTERSHEET_REFS}" (id 0) (at 230.8115 43.1006 0)
+    (property "Intersheet References" "${INTERSHEET_REFS}" (id 0) (at 233.0491 43.1006 0)
       (effects (font (size 1.27 1.27)) (justify right) hide)
     )
@@
   (global_label "RUMBLE+" (shape input) (at 88.9 76.2 180) (fields_autoplaced)
     (effects (font (size 1.27 1.27)) (justify right))
-    (property "Intersheet References" "${INTERSHEET_REFS}" (id 0) (at 77.5044 76.2794 0)
+    (property "Intersheet References" "${INTERSHEET_REFS}" (id 0) (at 77.5044 76.1206 0)
       (effects (font (size 1.27 1.27)) (justify right) hide)
     )
@@
   (symbol (lib_id "progcc_v3:SK6805-EC-15") (at 214.63 147.32 0) (unit 1)
     (in_bom yes) (on_board yes) (fields_autoplaced)
-    (property "Reference" "L4" (id 0) (at 214.63 137.16 0))
+    (property "Reference" "L6" (id 0) (at 214.63 137.16 0))
     (property "Value" "SK6805-EC-15" (id 1) (at 214.63 139.7 0))
     (property "Footprint" "progcc_v3:SK6805-EC-15" (id 2) (at 214.63 162.56 0)
@@
   (symbol (lib_id "progcc_v3:SK6805-EC-15") (at 191.77 147.32 0) (unit 1)
     (in_bom yes) (on_board yes) (fields_autoplaced)
-    (property "Reference" "L2" (id 0) (at 191.77 137.16 0))
+    (property "Reference" "L5" (id 0) (at 191.77 137.16 0))
     (property "Value" "SK6805-EC-15" (id 1) (at 191.77 139.7 0))
     (property "Footprint" "progcc_v3:SK6805-EC-15" (id 2) (at 191.77 162.56 0)
@@
   (symbol (lib_id "progcc_v3:SK6805-EC-15") (at 237.49 119.38 0) (unit 1)
     (in_bom yes) (on_board yes) (fields_autoplaced)
-    (property "Reference" "L5" (id 0) (at 237.49 109.22 0))
+    (property "Reference" "L3" (id 0) (at 237.49 109.22 0))
     (property "Value" "SK6805-EC-15" (id 1) (at 237.49 111.76 0))
     (property "Footprint" "progcc_v3:SK6805-EC-15" (id 2) (at 237.49 134.62 0)
@@
   (symbol (lib_id "progcc_v3:SK6805-EC-15") (at 260.35 119.38 0) (unit 1)
     (in_bom yes) (on_board yes) (fields_autoplaced)
-    (property "Reference" "L7" (id 0) (at 260.35 109.22 0))
+    (property "Reference" "L4" (id 0) (at 260.35 109.22 0))
     (property "Value" "SK6805-EC-15" (id 1) (at 260.35 111.76 0))
     (property "Footprint" "progcc_v3:SK6805-EC-15" (id 2) (at 260.35 134.62 0)
@@
   (symbol (lib_id "progcc_v3:SK6805-EC-15") (at 214.63 119.38 0) (unit 1)
     (in_bom yes) (on_board yes) (fields_autoplaced)
-    (property "Reference" "L3" (id 0) (at 214.63 109.22 0))
+    (property "Reference" "L2" (id 0) (at 214.63 109.22 0))
     (property "Value" "SK6805-EC-15" (id 1) (at 214.63 111.76 0))
     (property "Footprint" "progcc_v3:SK6805-EC-15" (id 2) (at 214.63 134.62 0)
@@
   (symbol (lib_id "progcc_v3:SK6805-EC-15") (at 237.49 147.32 0) (unit 1)
     (in_bom yes) (on_board yes) (fields_autoplaced)
-    (property "Reference" "L6" (id 0) (at 237.49 137.16 0))
+    (property "Reference" "L7" (id 0) (at 237.49 137.16 0))
     (property "Value" "SK6805-EC-15" (id 1) (at 237.49 139.7 0))
     (property "Footprint" "progcc_v3:SK6805-EC-15" (id 2) (at 237.49 162.56 0)
@@
       (reference "L1") (unit 1) (value "SK6805-EC-15") (footprint "progcc_v3:SK6805-EC-15")
     )
-    (path "/7fab03d3-d289-4ea6-8848-dbe6e72316a9"
+    (path "/c6420764-6844-4f7b-91d7-d916ab2d5614"
       (reference "L2") (unit 1) (value "SK6805-EC-15") (footprint "progcc_v3:SK6805-EC-15")
     )
-    (path "/c6420764-6844-4f7b-91d7-d916ab2d5614"
+    (path "/8b0d6696-0f7b-4e13-b84b-92fbaa37e0b4"
       (reference "L3") (unit 1) (value "SK6805-EC-15") (footprint "progcc_v3:SK6805-EC-15")
     )
-    (path "/5ef2d08d-60d6-42e5-b80d-d96d508d9ffa"
+    (path "/93a624cd-1ca1-45f9-abf4-c1e78faeac08"
       (reference "L4") (unit 1) (value "SK6805-EC-15") (footprint "progcc_v3:SK6805-EC-15")
     )
-    (path "/8b0d6696-0f7b-4e13-b84b-92fbaa37e0b4"
+    (path "/7fab03d3-d289-4ea6-8848-dbe6e72316a9"
       (reference "L5") (unit 1) (value "SK6805-EC-15") (footprint "progcc_v3:SK6805-EC-15")
     )
-    (path "/f28d5cca-96b0-4df9-8951-beec53bc4f20"
+    (path "/5ef2d08d-60d6-42e5-b80d-d96d508d9ffa"
       (reference "L6") (unit 1) (value "SK6805-EC-15") (footprint "progcc_v3:SK6805-EC-15")
     )
-    (path "/93a624cd-1ca1-45f9-abf4-c1e78faeac08"
+    (path "/f28d5cca-96b0-4df9-8951-beec53bc4f20"
       (reference "L7") (unit 1) (value "SK6805-EC-15") (footprint "progcc_v3:SK6805-EC-15")
     )

Commit message: some positioning changes+fP adjustments
Parts:
- added J1, J2: Rumble, progcc_v3:rumble_pins, symbol Connector:Conn_01x02_Male
- C5, C6, C7: footprint Capacitor_SMD:C_0603_1608Metric_Pad1.08x0.95mm_HandSolder -> Capacitor_SMD:C_0402_1005Metric
- JP1, JP2: footprint Jumper:SolderJumper-2_P1.3mm_Open_RoundedPad1.0x1.5mm -> Jumper:SolderJumper-2_P1.3mm_Open_TrianglePad1.0x1.5mm
- R20, R23, R24: footprint Resistor_SMD:R_0603_1608Metric_Pad0.98x0.95mm_HandSolder -> Resistor_SMD:R_0402_1005Metric
Connections:
- net +5V: now also J1.1 (Pin_1), J2.1 (Pin_1)
- net GND: no longer J9.S1 (SHIELD)
- net RUMBLE-: now also J1.2 (Pin_2), J2.2 (Pin_2)

Commit message: major routing
most of the board is routed minus a couple bits
Connections:
- net +3.3V is gone; now on net +3V3: C6.1, C7.1, Q4.1 (G), Q5.1 (G), Q6.1 (G), R10.1, R20.1, R6.1, R7.1, U1.1 (VDD), U2.1 (VDD), U3.1 (VDD), U4.1 (VDD), U5.1 (VDD)

Commit message: Kicad 7 and Routing
More routing done
Updated to Kicad 7 file types
Parts:
- removed C14, C16, C20, C23: 100n, Capacitor_SMD:C_0402_1005Metric, symbol Device:C
- removed C15: 1u, Capacitor_SMD:C_0402_1005Metric, symbol Device:C
- removed TP10, TP12: TestPoint, TestPoint:TestPoint_Pad_D1.5mm, symbol Connector:TestPoint
- added J5: Conn_01x02_Pin, Connector_PinHeader_2.00mm:PinHeader_1x02_P2.00mm_Vertical, symbol Connector:Conn_01x02_Pin
- R1, R15, R16, R17, R18, R2, R3, R4, R5: footprint Resistor_SMD:R_0603_1608Metric_Pad0.98x0.95mm_HandSolder -> Resistor_SMD:R_0402_1005Metric
- R21: footprint Resistor_SMD:R_0603_1608Metric_Pad0.98x0.95mm_HandSolder -> Resistor_SMD:R_0402_1005Metric_Pad0.72x0.64mm_HandSolder
Connections:
- net GULI_DAT is gone; now on net GULI_CALIBRATE: C5.1
- net LS_BUTTON: now also U6.14 (GPIO11)
- net RS_BUTTON: now also U6.13 (GPIO10)
- net UART0_TX: now reaches U6.15 (GPIO12)
- net UART0_TX: now also J5.1 (Pin_1)
- net UART0_RX: now reaches U6.16 (GPIO13)
- net UART0_RX: now also J5.2 (Pin_2)
Other:
- note added: "UART0 Debug"
- moved on the sheet: C13, C21, C22
